File: 36V 3.6A 30D/DEV-BOARD/Hardware/PowerServo AE 36V 3.6A 30D - DEV.kicad_sch (KiCad schematic)
At the start: 27 parts, among them IC1 DRV8251DDAR, J1 Control_In, J2 MOT_A, J3 Prog_IN, J4 Power_In, J6 Control_In, J7 MOT_B, U1 LMZM23601V5, U2 TLV76733DRVx, U4 MA730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

Commit message: Dev Version for Tests
Parts:
- removed J3: Prog_IN, Connector_PinHeader_1.27mm:PinHeader_2x03_P1.27mm_Vertical, symbol Connector_Generic:Conn_02x03_Odd_Even
- added J10: Debug_IN1, Connector_PinHeader_1.27mm:PinHeader_1x01_P1.27mm_Vertical, symbol Connector:Conn_01x01_Pin
- added J11: Debug_IN2, Connector_PinHeader_1.27mm:PinHeader_1x01_P1.27mm_Vertical, symbol Connector:Conn_01x01_Pin
- added J12: Debug_ISEN, Connector_PinHeader_1.27mm:PinHeader_1x01_P1.27mm_Vertical, symbol Connector:Conn_01x01_Pin
- added J13: Debug_VREF, Connector_PinHeader_1.27mm:PinHeader_1x01_P1.27mm_Vertical, symbol Connector:Conn_01x01_Pin
- added J16: Debug_5V, Connector_PinHeader_1.27mm:PinHeader_1x01_P1.27mm_Vertical, symbol Connector:Conn_01x01_Pin
- added J17: Debug_3.3V, Connector_PinHeader_1.27mm:PinHeader_1x01_P1.27mm_Vertical, symbol Connector:Conn_01x01_Pin
- added J3: Conn_02x07_Odd_Even, Connector_PinHeader_1.27mm:PinHeader_2x07_P1.27mm_Vertical, symbol Connector_Generic:Conn_02x07_Odd_Even
- added J5: Control_In, Connector_JST:JST_XH_B2B-XH-A_1x02_P2.50mm_Vertical, symbol Connector_Generic:Conn_01x02
- added J8: PWM/PWR, Connector_JST:JST_XH_B3B-XH-A_1x03_P2.50mm_Vertical, symbol Connector_Generic:Conn_01x03
- added J9: Debug_PWM_IN, Connector_PinHeader_1.27mm:PinHeader_1x01_P1.27mm_Vertical, symbol Connector:Conn_01x01_Pin
- IC1: footprint SOIC127P600X170-9N -> _custom:SOIC127P600X170-9N
Connections:
- net +3V3: now also J13.1 (Pin_1), J17.1 (Pin_1), J3.3 (Pin_3), J8.1 (Pin_1)
- net +5V: now also J16.1 (Pin_1)
- net DRV_IN1: now also J10.1 (Pin_1)
- net DRV_IN2: now also J11.1 (Pin_1)
- net GND: now also J3.11 (Pin_11), J3.5 (Pin_5), J3.7 (Pin_7), J8.3 (Pin_3)
- net ISEN: now also J12.1 (Pin_1)
- net NRST: now also J3.12 (Pin_12)
- net SWCLK: now also J3.6 (Pin_6)
- net SWDIO: now also J3.4 (Pin_4)
- net uC_UART_TX: now reaches U7.19 (PA9/UCPD1_DBCC1)
- net uC_UART_TX: now also J5.1 (Pin_1)
- net uC_UART_RX: now reaches U7.21 (PA10/UCPD1_DBCC2)
- net uC_UART_RX: now also J5.2 (Pin_2)
- net uC_PWM_IN: now reaches U7.22 (PA11/PA9)
- net uC_PWM_IN: now also J8.2 (Pin_2), J9.1 (Pin_1)
- no-connect marks 10 -> 17
Other:
- note added: "PWM_IN"
- note added: "USART"
- moved on the sheet: C10, R1, R3
